Commit message: added an IMU for the robot

File: description/gazebo_sensors.xacro (robot description, xacro)
@@ -95,3 +95,16 @@
         </sensor>
     </gazebo>
+    <!-- =========================================== -->
+    <!-- =============== IMU SENSOR ================= -->
+    <!-- =========================================== -->
+    <gazebo reference="imu_link">
+        <sensor name="imu_sensor" type="imu">
+            <pose>0 0 0 0 0 0</pose>
+            <always_on>true</always_on>
+            <visualize>true</visualize>
+            <update_rate>100</update_rate>
+            <topic>imu</topic>
+            <gz_frame_id>imu_link</gz_frame_id>
+        </sensor>
+    </gazebo>
 </robot>

File: description/joints.xacro (robot description, xacro)
@@ -82,3 +82,11 @@
         <origin xyz="0 0 0.05" rpy="0 0 0"/>
     </joint>
+    <!-- =========================================== -->
+    <!-- =============== IMU JOINT ================== -->
+    <!-- =========================================== -->
+    <joint name="imu_joint" type="fixed">
+        <parent link="base_link"/>
+        <child link="imu_link"/>
+        <origin xyz="0 0 0.175" rpy="0 0 0"/>
+    </joint>
 </robot>

File: description/links.xacro (robot description, xacro)
@@ -188,3 +188,22 @@
         </xacro:inertial_cylinder>
     </link>
+    <!-- =========================================== -->
+    <!-- ================ IMU LINK ================== -->
+    <!-- =========================================== -->
+    <link name="imu_link">
+        <visual>
+            <geometry>
+                <box size="0.025 0.025 0.025"/>
+            </geometry>
+            <material name="red"/>
+        </visual>
+        <collision>
+            <geometry>
+                <box size="0.025 0.025 0.025"/>
+            </geometry>
+        </collision>
+        <xacro:inertial_box mass="0.1" x="0.025" y="0.025" z="0.025">
+            <origin xyz="0 0 0" rpy="0 0 0"/>
+        </xacro:inertial_box>
+    </link>
 </robot>

Commit message: added GPS to the project

File: description/gazebo_sensors.xacro (robot description, xacro)
@@ -108,3 +108,14 @@
         </sensor>
     </gazebo>
+    <!-- =========================================== -->
+    <!-- =============== GPS SENSOR ================= -->
+    <!-- =========================================== -->
+    <gazebo reference="gps_link">
+        <sensor name="navsat_sensor" type="navsat">
+            <always_on>true</always_on>
+            <update_rate>5</update_rate>
+            <topic>gps/fix</topic>
+            <gz_frame_id>gps_link</gz_frame_id>
+        </sensor>
+    </gazebo>
 </robot>

File: description/joints.xacro (robot description, xacro)
@@ -83,5 +83,5 @@
     </joint>
     <!-- =========================================== -->
-    <!-- =============== IMU JOINT ================== -->
+    <!-- =============== IMU JOINT ================= -->
     <!-- =========================================== -->
     <joint name="imu_joint" type="fixed">
@@ -90,3 +90,11 @@
         <origin xyz="0 0 0.175" rpy="0 0 0"/>
     </joint>
+    <!-- =========================================== -->
+    <!-- ============== GPS JOINT ================== -->
+    <!-- =========================================== -->
+    <joint name="gps_joint" type="fixed">
+        <parent link="base_link"/>
+        <child link="gps_link"/>
+        <origin xyz="0 0 0.175" rpy="0 0 0"/>
+    </joint>
 </robot>

File: description/links.xacro (robot description, xacro)
@@ -207,3 +207,22 @@
         </xacro:inertial_box>
     </link>
+    <!-- =========================================== -->
+    <!-- ================ IMU LINK ================== -->
+    <!-- =========================================== -->
+    <link name="gps_link">
+        <visual>
+            <geometry>
+            <cylinder radius="0.02" length="0.02"/>
+            </geometry>
+            <material name="gray"/>
+        </visual>
+        <collision>
+            <geometry>
+                <cylinder radius="0.02" length="0.02"/>
+            </geometry>
+        </collision>
+        <xacro:inertial_cylinder mass="0.05" length="0.02" radius="0.02">
+            <origin xyz="0 0 0" rpy="0 0 0"/>
+        </xacro:inertial_cylinder>
+    </link>
 </robot>
